File: hardware/HT07/HT07.sch (KiCad schematic (older format))
At the start: 35 parts, among them J30 Conn_02x04_Odd_Even, P1 Conn_01x01_MountingPin, P2 Conn_01x01_MountingPin, P3 Conn_01x01_MountingPin, P4 Conn_01x01_MountingPin, SW30 SW_Push, U1 HDC2021, U2 NT3H2111W0FTTJ, U3 MSP430FR2155TDBT, U4 SIP32431DR3-T1GE3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

Commit message: HT07R2 sent to manufacture at Eurocircuits
Parts:
- R3: value 47K -> 100K; MANF PANASONIC -> BOURNS; MANF# ERJ2RKF4702X -> CR0402-FX-1003GLF; SUPPLIER FARNELL -> MOUSER; SUPPLIER# 2302806 -> 652-CR0402FX-1003GLF
Connections:
- no-connect marks 5 -> 27
Changed lines of the file:
@@
 AR Path="/6071CD30" Ref="R3"  Part="1"
 F 0 "R3" V 4080 4550 50  0000 C CNN
-F 1 "47K" V 4000 4550 50  0000 C CNN
+F 1 "100K" V 4000 4550 50  0000 C CNN
 F 2 "CUPL_FP:R_0402_1005Metric" V 3930 4550 50  0001 C CNN
 F 3 "" H 4000 4550 50  0001 C CNN
-F 4 "PANASONIC" H 4000 4550 50  0001 C CNN "MANF"
-F 5 "ERJ2RKF4702X" H 4000 4550 50  0001 C CNN "MANF#"
-F 6 "FARNELL" H 4000 4550 50  0001 C CNN "SUPPLIER"
-F 7 "2302806" H 4000 4550 50  0001 C CNN "SUPPLIER#"
+F 4 "BOURNS" H 4000 4550 50  0001 C CNN "MANF"
+F 5 "CR0402-FX-1003GLF" H 4000 4550 50  0001 C CNN "MANF#"
+F 6 "MOUSER" H 4000 4550 50  0001 C CNN "SUPPLIER"
+F 7 "652-CR0402FX-1003GLF" H 4000 4550 50  0001 C CNN "SUPPLIER#"
 	1    4000 4550
 	1    0    0    -1
@@
 EndData
 $EndBitmap
+NoConn ~ 10200 950
+NoConn ~ 10200 1050
+NoConn ~ 10200 1150
+NoConn ~ 10200 1250
+NoConn ~ 10200 1450
+NoConn ~ 10200 1550
+NoConn ~ 10200 1650
+NoConn ~ 10200 1750
+NoConn ~ 10200 2050
+NoConn ~ 10200 2150
+NoConn ~ 10200 2250
+NoConn ~ 10200 2350
+NoConn ~ 10200 2450
+NoConn ~ 10200 2550
+NoConn ~ 10200 2650
+NoConn ~ 10200 2750
+NoConn ~ 7450 2750
+NoConn ~ 7450 2650
+NoConn ~ 7450 2550
+NoConn ~ 7450 2450
+NoConn ~ 7450 1150
+NoConn ~ 7450 1050
 $EndSCHEMATC

Commit message: Up-issued to Rev 3
This changes the humidity sensor to HDC2022 from HDC2021. Also adds alternate parts for the MSP430 and NT3H to the schematic.
Parts:
- U1: value HDC2021 -> HDC2022DEPR; MANF# HDC2021DEBT -> HDC2022DEPR; SUPPLIER# HDC2021DEBT -> HDC2022DEPR
- U2: ALT (none) -> ALT: NT3H2211W0FTTJ
- U3: ALT (none) -> ALT: MSP430FR2355TDBTR
Other:
- note removed: "See SLAA322D"
- note removed: "Set LFXTDRIVE=3"
Changed lines of the file:
@@
 Sheet 1 1
 Title "CUPL TAG"
-Date "2021-04-19"
-Rev "2"
+Date "2021-08-16"
+Rev "3"
 Comp "COPYRIGHT Plotsensor Ltd. 2021"
-Comment1 "Designed by Malcolm Mackay"
+Comment1 "https://github.com/cuplsensor/cupltag"
 Comment2 "Licenced under CERN OHL-v2-S"
-Comment3 "CUPL®"
+Comment3 "CUPL® Designed by Malcolm Mackay"
 Comment4 ""
 $EndDescr
@@
 P 6750 5550
 F 0 "U1" H 6550 5900 50  0000 R CNN
-F 1 "HDC2021" H 7050 5200 50  0000 R CNN
+F 1 "HDC2022DEPR" H 7250 5200 50  0000 R CNN
 F 2 "CUPL_FP:HDC2021" H 6750 5100 50  0001 C CNN
 F 3 "https://www.ti.com/lit/ds/symlink/hdc2021.pdf" H 6450 5850 50  0001 C CNN
 F 4 "TEXAS" H 6150 5000 60  0001 L CNN "MANF"
-F 5 "HDC2021DEBT" H 6500 4900 60  0001 C CNN "MANF#"
+F 5 "HDC2022DEPR" H 6500 4900 60  0001 C CNN "MANF#"
 F 6 "TEXAS" H 6300 4800 60  0001 C CNN "SUPPLIER"
-F 7 "HDC2021DEBT" H 6500 4700 60  0001 C CNN "SUPPLIER#"
+F 7 "HDC2022DEPR" H 6500 4700 60  0001 C CNN "SUPPLIER#"
 	1    6750 5550
 	1    0    0    -1
@@
 F 6 "FARNELL" H 8900 4600 60  0001 L CNN "SUPPLIER"
 F 7 "2663150" H 8900 4500 60  0001 L CNN "SUPPLIER#"
+F 8 "ALT: NT3H2211W0FTTJ" H 7850 4900 50  0000 L CNN "ALT"
 	1    8750 5350
 	-1   0    0    -1
@@
 	2300 1650 7450 1650
 $Comp
-L device:Battery_Cell BT30
-U 1 1 605C1351
-P 2000 4250
-F 0 "BT30" H 2118 4346 50  0000 L CNN
-F 1 "CR1220" H 2118 4255 50  0000 L CNN
-F 2 "CUPL_FP:MPD_BC501SM_CR1220" V 2000 4310 50  0001 C CNN
-F 3 "~" V 2000 4310 50  0001 C CNN
-F 4 "MPD" H 2000 4250 50  0001 C CNN "MANF"
-F 5 "BC501SM" H 2000 4250 50  0001 C CNN "MANF#"
-F 6 "DIGIKEY" H 2000 4250 50  0001 C CNN "SUPPLIER"
-F 7 "BC501SM-TRCT-ND" H 2000 4250 50  0001 C CNN "SUPPLIER#"
-	1    2000 4250
-	1    0    0    -1
-$EndComp
-$Comp
 L power:VDD #PWR0107
 U 1 1 605C3018
@@
 F 0 "C7" H 5925 1250 50  0000 L CNN
 F 1 "10U" H 5925 1050 50  0000 L CNN
-F 2 "CUPL_FP:C_0603_1608Metric" V 5700 1050 50  0000 C CNN
+F 2 "CUPL_FP:C_0603_1608Metric" H 5200 1150 50  0000 C CNN
 F 3 "" H 5900 1150 50  0000 C CNN
 F 4 "AVX" H 5900 1150 50  0001 C CNN "MANF"
@@
 Wire Wire Line
 	7350 1450 7350 5650
-Text Notes 5450 2750 0    60   ~ 0
-Set LFXTDRIVE=3
-Text Notes 5450 2850 0    60   ~ 0
-See SLAA322D
 Connection ~ 5950 1750
 Wire Wire Line
@@
 F 6 "MOUSER" H 7550 150 60  0001 L CNN "SUPPLIER"
 F 7 "595-MSP430FR2155TDBTR" H 7550 50  60  0001 L CNN "SUPPLIER#"
+F 8 "ALT: MSP430FR2355TDBTR" H 8050 500 50  0000 C CNN "ALT"
 	1    8850 1750
 	1    0    0    -1
@@
 NoConn ~ 7450 1150
 NoConn ~ 7450 1050
+$Comp
+L device:Battery_Cell BT30
+U 1 1 605C1351
+P 2000 4250
+F 0 "BT30" H 2118 4346 50  0000 L CNN
+F 1 "CR1220" H 2118 4255 50  0000 L CNN
+F 2 "CUPL_FP:MPD_BC501SM_CR1220" V 2000 4310 50  0001 C CNN
+F 3 "~" V 2000 4310 50  0001 C CNN
+F 4 "MPD" H 2000 4250 50  0001 C CNN "MANF"
+F 5 "BC501SM" H 2000 4250 50  0001 C CNN "MANF#"
+F 6 "DIGIKEY" H 2000 4250 50  0001 C CNN "SUPPLIER"
+F 7 "BC501SM-TRCT-ND" H 2000 4250 50  0001 C CNN "SUPPLIER#"
+	1    2000 4250
+	1    0    0    -1
+$EndComp
 $EndSCHEMATC

Commit message: Started to update documentation.
Parts:
- C10: SUPPLIER# 2781441 -> 2332495
Changed lines of the file:
@@
 F 5 "04025A180FAT2A" H 10100 5300 50  0001 C CNN "MANF#"
 F 6 "FARNELL" H 10100 5300 50  0001 C CNN "SUPPLIER"
-F 7 "2781441" H 10100 5300 50  0001 C CNN "SUPPLIER#"
+F 7 "2332495" H 10100 5300 50  0001 C CNN "SUPPLIER#"
 	1    10100 5300
 	-1   0    0    1
